Commit message: FIX: replace absolute paths

File: urdf/bittle.urdf (robot description, URDF)
Before this commit: robot bittle, 13 links, 12 joints
Links:
- link base-frame-link: mass 0.108 -> None; geometry collision mesh filename=package://champ_description_bittle/obj/base_frame.001.obj scale=1.0 1.0 1.0; visual mesh filename=package://champ_description_bittle/obj/base_frame.obj scale=1.0 1.0 1.0
- link battery-link: mass 0.056 -> None; geometry collision mesh filename=package://champ_description_bittle/obj/battery.001.obj scale=1.0 1.0 1.0; visual mesh filename=package://champ_description_bittle/obj/battery.obj scale=1.0 1.0 1.0
- link cover-link: mass 0.013 -> None; geometry collision mesh filename=package://champ_description_bittle/obj/cover.001.obj scale=1.0 1.0 1.0; visual mesh filename=package://champ_description_bittle/obj/cover.obj scale=1.0 1.0 1.0
- link imu_link: mass 0.001 -> None; geometry visual mesh filename=package://champ_description_bittle/obj/Cube.011.obj scale=1.0 1.0 1.0
- link left-back-knee-link: mass 0.017 -> None; geometry collision mesh filename=package://champ_description_bittle/obj/left_knee.002.obj scale=1.0 1.0 1.0; visual mesh filename=package://champ_description_bittle/obj/left_knee.001.obj scale=1.0 1.0 1.0
- link left-back-shoulder-link: mass 0.006 -> None; geometry collision mesh filename=package://champ_description_bittle/obj/shoulder.004.obj scale=1.0 1.0 1.0; visual mesh filename=package://champ_description_bittle/obj/shoulder.001.obj scale=1.0 1.0 1.0
- link left-front-knee-link: mass 0.017 -> None; geometry collision mesh filename=package://champ_description_bittle/obj/left_knee.003.obj scale=1.0 1.0 1.0; visual mesh filename=package://champ_description_bittle/obj/left_knee.obj scale=1.0 1.0 1.0
- link left-front-shoulder-link: mass 0.006 -> None; geometry collision mesh filename=package://champ_description_bittle/obj/shoulder.007.obj scale=1.0 1.0 1.0; visual mesh filename=package://champ_description_bittle/obj/shoulder.obj scale=1.0 1.0 1.0
- link mainboard_link: mass 0.001 -> None; geometry visual mesh filename=package://champ_description_bittle/obj/Plane.obj scale=1.0 1.0 1.0
- link right-back-knee-link: mass 0.017 -> None; geometry collision mesh filename=package://champ_description_bittle/obj/right_knee.002.obj scale=1.0 1.0 1.0; visual mesh filename=package://champ_description_bittle/obj/right_knee.001.obj scale=1.0 1.0 1.0
- link right-back-shoulder-link: mass 0.006 -> None; geometry collision mesh filename=package://champ_description_bittle/obj/shoulder.005.obj scale=1.0 1.0 1.0; visual mesh filename=package://champ_description_bittle/obj/shoulder.002.obj scale=1.0 1.0 1.0
- link right-front-knee-link: mass 0.017 -> None; geometry collision mesh filename=package://champ_description_bittle/obj/right_knee.003.obj scale=1.0 1.0 1.0; visual mesh filename=package://champ_description_bittle/obj/right_knee.obj scale=1.0 1.0 1.0
- link right-front-shoulder-link: mass 0.006 -> None; geometry collision mesh filename=package://champ_description_bittle/obj/shoulder.006.obj scale=1.0 1.0 1.0; visual mesh filename=package://champ_description_bittle/obj/shoulder.003.obj scale=1.0 1.0 1.0

Commit message: CHG: update URDF model to fit champ requiments

File: urdf/bittle.urdf (robot description, URDF)
Before this commit: robot bittle, 13 links, 12 joints
Links:
- added link left-back-foot-link; visual cylinder length=0.1 radius=0.02
- added link left-front-foot-link; visual cylinder length=0.1 radius=0.02
- added link right-back-foot-link; visual cylinder length=0.1 radius=0.02
- added link right-front-foot-link; visual cylinder length=0.1 radius=0.02
Joints:
- added joint left-back-foot-joint: type fixed, parent left-back-knee-link, child left-back-foot-link, origin xyz=0.01 -0.5 -0.1 rpy=0 0 0
- added joint left-front-foot-joint: type fixed, parent left-front-knee-link, child left-front-foot-link, origin xyz=0.01 -0.5 -0.1 rpy=0 0 0
- added joint right-back-foot-joint: type fixed, parent right-back-knee-link, child right-back-foot-link, origin xyz=0.01 -0.5 -0.1 rpy=0 0 0
- added joint right-front-foot-joint: type fixed, parent right-front-knee-link, child right-front-foot-link, origin xyz=0.01 -0.5 -0.1 rpy=0 0 0
